File: BUS REG, BA MUX.kicad_sch (KiCad schematic)
At the start: 10 parts

Commit message: updating to newest versions of schematics
Connections:
- net DAPB BAMX04 H: now also E5.7 (Y1)
- net DAPB BAMX05 H: now also E5.9 (Y2)
- net DAPB BMX04 H: now also E3.7 (Y1)
- net DAPB BMX05 H: now also E3.9 (Y2)
- net DAPB BNX00 H: now also E20.7 (Y1)
- net DAPB BNX01 H: now also E20.9 (Y2)
- net DAPB AMX00 H: now reaches E21.7 (Y1)
- net DAPA K0MX 02 H renamed DAPA K0MX02 H
- net DAPB BAMX 00 H renamed DAPB BAMX00 H
- net DAPD K0MX 00 H renamed DAPD K0MX00 H
- net DAPD K0MX 01 H renamed DAPD K0MX01 H
- net DAPD K1MX 01 H renamed DAPD K1MX01 H
- net DAPE BMXS1 LOB L renamed DAPB BMXS1 LOB L
- net DAPE K1MX 02 H renamed DAPE K1MX02 H
- net DAPE K1MX 03 H renamed DAPE K1MX03 H
- net DAPE K1MX 04 H renamed DAPE K1MX04 H
- net DAPE K1MX 05 H renamed DAPE K1MX05 H
