File: ALU, SHIFTER, PCA, PCB - PAGE 2.kicad_sch (KiCad schematic)
At the start: 13 parts

Commit message: updating to newest versions of schematics
Parts:
- removed unit 6 of E45
- renumbered E45 to E58
Connections:
- net DAPD AMX01 H is gone; now on net DAPC AMX08 H: E45.23 (A1)
- net GRAA ALUM L is gone; now on net GRAA ALUS1 L: E58.1
- net GRAA SFRS0 L is gone; now on net GRAA ALUS0 L: E58.11
- net DAPF ALU04 H: no longer E46.13 (D4)
- net DAPF ALU05 H: no longer E46.14 (D5)
- net DAPF ALU06 H: now also E46.3 (D0)
- net DAPF ALU07 H: now also E46.4 (D1)
- net DAPF COUT07 L: now also E45.7 (Cn)
- net DAPF LM H: no longer E45.8 (M), E58.6
- net DAPF LS0 H: no longer E45.6 (S0), E58.8
- net DAPF LS1 H: no longer E45.5 (S1), E58.2
- net DAPF LS2 H: no longer E45.4 (S2), E58.10
- net DAPF LS3 H: no longer E45.3 (S3)
- net DAPF PCB00 H: no longer E53.5 (1C1)
- net DAPF PCB01 H: no longer E53.11 (2C1)
- net DAPF PCB02 H: no longer E59.5 (1C1)
- net DAPF SHFRS0 H: no longer E59.14 (A)
- net DAPF SHFRS1 H: no longer E59.2 (B)
- net DAPH ALU08 H: now also E45.9 (F0), E46.6 (D2), E53.4 (1C2); no longer E53.6 (1C0)
- net DAPH ALU09 H: now also E45.10 (F1), E46.11 (D3), E53.12 (2C2), E53.3 (1C3); no longer E53.10 (2C0)
- net DAPH ALU10 H: now also E45.11 (F2), E46.13 (D4), E53.13 (2C3), E59.4 (1C2); no longer E59.6 (1C0)
- net DAPH ALU11 H: now also E45.13 (F3), E46.14 (D5), E59.12 (2C2), E59.3 (1C3)
- net GRAA ALUS0 L: no longer E58.9
- net GRAA ALUS1 L: no longer E58.5
- net at E45.15 (X): no longer E44.3 (G0)
- net at E45.17 (Y): no longer E44.4 (P0)
- net at E44.13 (Cn): no longer E45.7 (Cn)
- net DAPB AMX00 H renamed DAPC AMX08 H
- net DAPB BMX00 H renamed DAPC BMX08 H
- net DAPB BMX01 H renamed DAPC BMX09 H
- net DAPB BMX02 H renamed DAPC BMX10 H
- net DAPB BMX03 H renamed DAPC BMX11 H
- net DAPD AMX02 H renamed DAPC AMX10 H
- net DAPD AMX03 H renamed DAPC AMX11 H
- removed net DAPF ALU08 H: E45.9 (F0), E46.3 (D0), E53.12 (2C2), E53.4 (1C2)
- removed net DAPF ALU09 H: E45.10 (F1), E46.4 (D1), E53.13 (2C3), E53.3 (1C3)
- removed net DAPF ALU10 H: E45.11 (F2), E46.6 (D2), E59.4 (1C2)
- removed net DAPF ALU11 H: E45.13 (F3), E46.11 (D3), E59.12 (2C2), E59.3 (1C3)
- new net DAPF ALU00 H: E53.6 (1C0)
- new net DAPF ALU01 H: E53.10 (2C0)
- new net DAPF ALU02 H: E59.6 (1C0)
- new net DAPH HM H: E45.8 (M)
- new net DAPH HS0 H: E45.6 (S0), E58.10
- new net DAPH HS1 H: E45.5 (S1), E58.2
- new net DAPH HS2 H: E45.4 (S2), E58.8
- new net DAPH HS3 H: E45.3 (S3), E58.6
- new net DAPH PCB08 H: E53.5 (1C1)
- new net DAPH PCB09 H: E53.11 (2C1)
- new net DAPH PCB10 H: E59.5 (1C1)
- new net GRAA ALUS2 L: E58.9
- new net GRAA ALUS3 L: E58.5
Other:
- note removed: "NEED TO SWAP THESE PORTS AND NETS TO PAGE 37"
- moved on the sheet: E44

Commit message: Fixed net labels and added caps to BOM
Parts:
- removed E43, E58, E59, E79: 74LS04, symbol 74xx:74LS04
- removed E44, E49: 74LS182, symbol 74xx:74LS182
- removed E45, E48: 74LS181, Package_DIP:DIP-24_18.0mmx34.29mm_W15.24mm, symbol 74xx:74LS181
- removed E46, E47: 74LS174, symbol 74xx:74LS174
- removed E53, E81, E82: 74S153, DIP16, symbol Untitled-altium-import:root_0_74S153
Connections:
- no-connect marks 10 -> 0
