File: trap_vectors.kicad_sch (KiCad schematic)
At the start: 24 parts

Commit message: Fixed net labels and added caps to BOM
Parts:
- added C1, C2, C3, C?: 6.8uF, Capacitor_THT:C_Rect_L7.5mm_W6.5mm_P5.00mm, symbol Device:C_Polarized
Connections:
- net +5: now also C1.1, C2.1, C3.1, C?.1
- net DAPE K1EX H: now also E25.9 (Y2)
- net DAPE K1MX01 H: now also E9.7 (Y1)
- net DAPE K1MX02 H: now also E9.9 (Y2)
- net DAPE K1MX03 H: now also E19.7 (Y1)
- net DAPE K1MX04 H: now also E19.9 (Y2)
- net DAPE K1MX05 H: now also E24.7 (Y1)
- net DAPE K1MX06 H: now also E24.9 (Y2)
- net DAPE K1MX07 H: now also E25.7 (Y1)
- net DAPE SV02 H: now also E18.12 (6Y)
- net DAPE SV03 H: now also E18.10 (5Y)
- net DAPE SV04 H: now also E17.8 (4Y)
- net DAPE SV05 H: now also E18.6 (3Y)
- net DAPE SV06 H: now also E18.4 (1Y)
- net DAPE SV07 H: now also E18.2 (1Y)
- net DAPE TV03 H: now also E8.6 (Y2)
- net DAPE TV04 H: now also E16.8 (Y3)
- net DAPE TV05*07 H: now also E16.6 (Y2)
